File: Elétrica/glicosimetro/glicosimetro.kicad_sch (KiCad schematic)
At the start: 15 parts, among them U1 ESP32-C3_SUPERMINI, U2 MCP6004, U3 OPA2381, U4 LM1117DT-3.3, U5 CD4051B

Commit message: Atualizações
Parts:
- removed D1: S5971, OptoDevice:Osram_BPW34S-SMD, symbol Sensor_Optical:BPW34-SMD
- removed U2: MCP6004, symbol Amplifier_Operational:MCP6004
- removed U3: OPA2381, Package_SO:SOIC-8_3.9x4.9mm_P1.27mm, symbol Amplifier_Operational:OPA2340
- removed U5: CD4051B, MUX:DIP794W45P254L1969H508Q16, symbol Analog_Switch:CD4051B
- added C5: 0.1uF, Capacitor_SMD:C_0603_1608Metric_Pad1.08x0.95mm_HandSolder, symbol Device:C
- added C6, C7, C8: C, Capacitor_SMD:C_0603_1608Metric_Pad1.08x0.95mm_HandSolder, symbol Device:C
- added D1: MTE8120CP 805nm, LED_SMD:LED_1206_3216Metric, symbol LED:IR26-21C_L110_TR8
- added Q1, Q2: BC337, Package_TO_SOT_THT:TO-92_Inline, symbol Transistor_BJT:BC337
- added R1, R2, R3, R6, R7, R8, R9: R, Resistor_SMD:R_0603_1608Metric, symbol Device:R
- added U3: MCP6002-xMC, Package_DFN_QFN:DFN-8-1EP_3x2mm_P0.5mm_EP1.75x1.45mm, symbol Amplifier_Operational:MCP6002-xMC
- added U6: MCP601R, Package_TO_SOT_SMD:SOT-23-5, symbol Amplifier_Operational:MCP601R
- added U7: LTC6910-1CTS8PBF, LTC6910-1CTS8PBF:SOT65P280X100-8N, symbol LTC6910-1CTS8PBF:LTC6910-1CTS8PBF
- C1: value 1uF -> C
- R4, R5: value 27R -> R; footprint Resistor_SMD:R_0603_1608Metric_Pad0.98x0.95mm_HandSolder -> Resistor_SMD:R_0603_1608Metric
Connections:
- net BIT_1 is gone; now on net LED1: U1.8 (GPIO8)
- net 3v3: now also D2.2 (A), C5.1, D1.2 (A), U3.8 (V+), U6.5 (V+), U7.8 (V+)
- net GND: now also C5.2, Q1.3 (E), Q2.3 (E), R7.1, U3.2 (-), U3.4 (V-), U3.5 (+), U3.9 (V-), U6.2 (V-), U6.3 (+), U7.2 (AGND), U7.4 (V-); no longer D2.1 (K), D3.1 (K)
- net LED2: now also U1.9 (GPIO9)
- net at C2.1, D4.1 (K): now also R2.1, U6.4 (-)
- net at D3.2 (A): no longer R5.2
- net at C1.1: now also R3.2, U3.3 (+)
- net at R4.2: now also Q1.2 (B); no longer D2.2 (A)
- net LTC_B0: now reaches U1.10 (GPIO10)
- net LTC_B0: now also U7.5 (G0)
- net LTC_B1: now reaches U1.20 (GPIO20)
- net LTC_B1: now also U7.6 (G1)
- net LTC_B2: now reaches U1.21 (GPIO21)
- net LTC_B2: now also U7.7 (G2)
- net PF - entrada AD: now reaches U1.5 (GPIO5)
- net PF - entrada AD: now also R6.2, U3.7
- net BIT_0: no longer names the net of U1.7 (GPIO7)
- net IN_AD renamed PB - entrada AD
- net PB - entrada AD: now also C6.2, C8.1, U3.1
- new net: D1.1 (K), R8.2
- new net: Q1.1 (C), R8.1
- new net: Q2.1 (C), R9.1
- new net: D2.1 (K), R9.2
- new net: C7.1, C8.2, R6.1
- new net: C6.1, R1.2, R3.1
- new net: Q2.2 (B), R5.2
- new net: C7.2, R7.2, U3.6 (-)
- new net Estágio 2_Ganho: R2.2, U6.1, U7.3 (IN)
- new net Estágio3_Filtro: R1.1, U7.1 (OUT)
- no-connect marks 5 -> 6
Other:
- note added: "1"
- note added: "2"
- note added: "3"
- note added: "AMPLIFICADOR DE TRANSIMPEDÂNCIA"
- note added: "CAPTURA DE SINAL"
- note added: "CONTROLADOR"
- note added: "GANHO PROGRAMÁVEL"
- note added: "PASSA ALTA"
- note added: "PASSA BAIXA"
- note added: "REGULADOR DE TENSÃO"
- note removed: "RNCF1206TKW27R0"
- moved on the sheet: C2, C3, C4, D2, D3, D4, U1, U4
