File: Elétrica/Glicosímetro para cablibração/gluco_calibration/gluco_calibration.kicad_sch (KiCad schematic)
At the start: 28 parts, among them J1 Conn_01x15, J2 Conn_01x15, J3 Conn_01x15, J4 Conn_01x15, Q1 BC337, Q2 BC337, U1 MCP6002-xMC, U2 MCP602

Commit message: transimpedancia
mudei a entrada para a inversora
Connections:
- net Vref: now also U2.3 (+); no longer U2.2 (-)
- net at C5.1, D4.1 (K), R5.1: now also U2.2 (-); no longer U2.3 (+)
Changed lines of the file:
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@@
+	)
+	(junction
+		(at 139.7 39.37)
+		(diameter 0)
+		(color 0 0 0 0)
 	)
 	(junction
@@
 	)
 	(junction
-		(at 146.05 34.29)
-		(diameter 0)
-		(color 0 0 0 0)
-	)
-	(junction
 		(at 44.45 92.71)
 		(diameter 0)
@@
 	(wire
 		(pts
-			(xy 157.48 25.4) (xy 146.05 25.4)
+			(xy 157.48 25.4) (xy 139.7 25.4)
 		)
 		(stroke
@@
 	(wire
 		(pts
-			(xy 139.7 34.29) (xy 139.7 53.34)
-		)
-		(stroke
-			(width 0)
-			(type default)
-		)
-	)
-	(wire
-		(pts
 			(xy 96.52 40.64) (xy 96.52 55.88)
 		)
@@
 	(wire
 		(pts
+			(xy 152.4 34.29) (xy 153.67 34.29)
+		)
+		(stroke
+			(width 0)
+			(type default)
+		)
+	)
+	(wire
+		(pts
 			(xy 74.93 76.2) (xy 74.93 95.25)
 		)
@@
 	(wire
 		(pts
-			(xy 139.7 34.29) (xy 146.05 34.29)
-		)
-		(stroke
-			(width 0)
-			(type default)
-		)
-	)
-	(wire
-		(pts
 			(xy 69.85 25.4) (xy 50.8 25.4)
 		)
@@
 	(wire
 		(pts
-			(xy 149.86 39.37) (xy 153.67 39.37)
-		)
-		(stroke
-			(width 0)
-			(type default)
-		)
-	)
-	(wire
-		(pts
 			(xy 149.86 104.14) (xy 149.86 105.41)
 		)
@@
 	(wire
 		(pts
+			(xy 139.7 39.37) (xy 139.7 53.34)
+		)
+		(stroke
+			(width 0)
+			(type default)
+		)
+	)
+	(wire
+		(pts
+			(xy 139.7 39.37) (xy 153.67 39.37)
+		)
+		(stroke
+			(width 0)
+			(type default)
+		)
+	)
+	(wire
+		(pts
 			(xy 95.25 55.88) (xy 96.52 55.88)
 		)
@@
 	(wire
 		(pts
-			(xy 146.05 34.29) (xy 153.67 34.29)
-		)
-		(stroke
-			(width 0)
-			(type default)
-		)
-	)
-	(wire
-		(pts
 			(xy 165.1 25.4) (xy 170.18 25.4)
 		)
@@
 	(wire
 		(pts
-			(xy 146.05 25.4) (xy 146.05 34.29)
+			(xy 139.7 25.4) (xy 139.7 39.37)
 		)
 		(stroke
@@
 	(global_label "Vref"
 		(shape input)
-		(at 149.86 39.37 270)
-		(fields_autoplaced yes)
-		(effects
-			(font
-				(size 1.27 1.27)
-			)
-			(justify right)
-		)
-		(property "Intersheetrefs" "${INTERSHEET_REFS}"
-			(at 149.86 46.0443 90)
-			(effects
-				(font
-					(size 1.27 1.27)
-				)
-				(justify right)
-				(hide yes)
-			)
+		(at 152.4 34.29 90)
+		(fields_autoplaced yes)
+		(effects
+			(font
+				(size 1.27 1.27)
+			)
+			(justify left)
+		)
+		(property "Intersheetrefs" "${INTERSHEET_REFS}"
+			(at 152.4 27.6157 90)
+			(effects
+				(font
+					(size 1.27 1.27)
+				)
+				(justify left)
+				(hide yes)
+			)

Commit message: trab para apresentação
Connections:
- net Vref: now also D4.1 (K); no longer D4.2 (A)
- net at C5.1, R5.1, U2.2 (-): now also D4.2 (A); no longer D4.1 (K)
Other:
- moved on the sheet: D4
Changed lines of the file:
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@@
 	(wire
 		(pts
-			(xy 133.35 63.5) (xy 133.35 62.23)
-		)
-		(stroke
-			(width 0)
-			(type default)
-		)
-	)
-	(wire
-		(pts
 			(xy 96.52 40.64) (xy 96.52 55.88)
 		)
@@
 	(wire
 		(pts
-			(xy 146.05 63.5) (xy 146.05 62.23)
+			(xy 146.05 62.23) (xy 146.05 64.77)
 		)
 		(stroke
@@
 	(wire
 		(pts
+			(xy 133.35 53.34) (xy 133.35 57.15)
+		)
+		(stroke
+			(width 0)
+			(type default)
+		)
+	)
+	(wire
+		(pts
 			(xy 57.15 92.71) (xy 53.34 92.71)
 		)
@@
 	(wire
 		(pts
-			(xy 133.35 53.34) (xy 133.35 54.61)
-		)
-		(stroke
-			(width 0)
-			(type default)
-		)
-	)
-	(wire
-		(pts
-			(xy 133.35 63.5) (xy 146.05 63.5)
-		)
-		(stroke
-			(width 0)
-			(type default)
-		)
-	)
-	(wire
-		(pts
 			(xy 69.85 25.4) (xy 50.8 25.4)
 		)
@@
 	(wire
 		(pts
+			(xy 146.05 64.77) (xy 133.35 64.77)
+		)
+		(stroke
+			(width 0)
+			(type default)
+		)
+	)
+	(wire
+		(pts
 			(xy 139.7 53.34) (xy 146.05 53.34)
 		)
@@
 	(global_label "Vref"
 		(shape input)
-		(at 139.7 63.5 270)
+		(at 139.7 64.77 270)
 		(fields_autoplaced yes)
 		(effects
@@
 		)
 		(property "Intersheetrefs" "${INTERSHEET_REFS}"
-			(at 139.7 70.1743 90)
+			(at 139.7 71.4443 90)
 			(effects
 				(font
@@
 	(symbol
 		(lib_id "Sensor_Optical:BPW34")
-		(at 133.35 59.69 270)
+		(at 133.35 59.69 90)
 		(unit 1)
 		(exclude_from_sim no)
@@
 		(dnp no)
 		(property "Reference" "D4"
-			(at 127 57.658 90)
+			(at 139.7 61.722 90)
 			(effects
 				(font
@@
 		)
 		(property "Value" "BPW34"
-			(at 124.714 59.436 90)
+			(at 141.986 59.944 90)
 			(effects
 				(font
@@
 		)
 		(property "Footprint" "OptoDevice:Osram_DIL2_4.3x4.65mm_P5.08mm"
-			(at 137.795 59.69 0)
+			(at 128.905 59.69 0)
 			(effects
 				(font
@@
 		)
 		(property "Datasheet" "http://www.vishay.com/docs/81521/bpw34.pdf"
-			(at 133.35 58.42 0)
+			(at 133.35 60.96 0)
 			(effects
 				(font
